Commit message: Update URDFPRUEBA2.urdf
Corregido y funcional en los ejes

File: Modelos Simulacion/URDFPRUEBA2.urdf (robot description, URDF)
Before this commit: robot robot, 4 links, 3 joints
Joints:
- joint link_1_joint: origin xyz=0 0 0 rpy=0 0 0 -> xyz=0.12 0 0 rpy=0 0 0
- joint link_2_joint: origin xyz=0 0 0 rpy=0 0 0 -> xyz=0.083 0 0 rpy=0 0 0
- joint link_3_joint: origin xyz=0 0 0 rpy=0 0 0 -> xyz=0.195 0 0 rpy=0 0 0
