Commit message: Add files via upload

File: hexapod_description/urdf/hexapod_description.urdf (robot description, URDF)
Before this commit: robot hexapod_description, 19 links, 18 joints
Links:
- link 1A_link: mass 0.0263699504711605 -> 0.0284343546565839
- link 1B_link: mass 0.0393326462006014 -> 0.0393326462004403
- link 2A_link: mass 0.0263699508381395 -> 0.0284343550237236
- link 2B_link: mass 0.0393326465544563 -> 0.0393326465544562
- link 2C_link: mass 0.0544820458081965 -> 0.0544820458081966
- link 3A_link: mass 0.0263699508285937 -> 0.0284343550141747
- link 3B_link: mass 0.0393326465589695 -> 0.0393326465589664
- link 3C_link: mass 0.0544820458081964 -> 0.0544820458081965
- link 4A_link: mass 0.0263699504710962 -> 0.0284343546567147
- link 4B_link: mass 0.0393326462005431 -> 0.0393326462005796
- link 4C_link: mass 0.0544820458081964 -> 0.0544820458081965
- link 5A_link: mass 0.0263699508381523 -> 0.0284343550237688
- link 5B_link: mass 0.0393326465544562 -> 0.0393326465544563
- link 5C_link: mass 0.0544820458081966 -> 0.0544820458081965
- link 6A_link: mass 0.0263699508285987 -> 0.0284343550141806
- link 6B_link: mass 0.039332646558969 -> 0.039332646558968
- link base_link: mass 0.406550708950941 -> 0.394164283837447
Joints:
- joint 1A_joint: axis 0 0 0.999999999991391 -> 0 0 1; origin xyz=-0.260544565013545 -1.01206116241563 -0.281391297394327 rpy=-1.5707963267949 1.49476626971651 -3.14159265358979 -> xyz=-0.26054 -1.0121 -0.28139 rpy=-1.5708 1.4948 -3.1416
- joint 1B_joint: axis -0.0449475329048584 -0.0503765997912149 -0.997718355789469 -> -0.044948 -0.050377 -0.99772; origin xyz=0.0636203974674808 -0.000577139628543943 0.00570103050496762 rpy=1.57080045971871 0.842287346673303 3.13252412666513 -> xyz=0.06362 -0.00057714 0.005701 rpy=1.5708 0.84229 3.1325
- joint 1C_joint: axis -0.0102179351134587 -0.99771835169199 -0.0667359310943994 -> -0.010218 -0.99772 -0.066736; origin xyz=-0.164084019172298 -0.00845892892413586 -0.0272391911814598 rpy=1.57079626680283 0 2.26115671183903 -> xyz=-0.16408 -0.0084589 -0.027239 rpy=1.5708 0 2.2612
- joint 2A_joint: axis 0 0 0.999999999991391 -> 0 0 1; origin xyz=-0.378260308632601 -1.03316169228736 -0.209825331186314 rpy=-1.5707963267949 0.447803456724678 -3.14159265358979 -> xyz=-0.37826 -1.0332 -0.20983 rpy=-1.5708 0.4478 -3.1416
- joint 2B_joint: axis 0.0328663838674289 0.0587298554671745 -0.997732732192486 -> 0.032866 0.05873 -0.99773; origin xyz=0.0635994650152483 -0.000578393068543129 -0.0153999472755177 rpy=-1.57080465259821 -1.06059839350069 -0.00908580645889822 -> xyz=0.063599 -0.00057839 -0.0154 rpy=-1.5708 -1.0606 -0.0090858
- joint 2C_joint: axis 0.0618783699585716 0.997732286459228 0.0264830490712859 -> 0.061878 0.99773 0.026483; origin xyz=0.171099091710239 0 0.00973951247489032 rpy=-1.57079893258156 0 0.656200837708118 -> xyz=0.1711 0 0.0097395 rpy=-1.5708 0 0.6562
- joint 3A_joint: axis 0 0 0.999999999991391 -> 0 0 1; origin xyz=-0.374914944478911 -1.03316214363253 -0.071745054027157 rpy=-1.5707963267949 -0.633602285574073 3.14159265358979 -> xyz=-0.37491 -1.0332 -0.071745 rpy=-1.5708 -0.6336 3.1416
- joint 3B_joint: axis 0.0409633277318722 0.0929442335923958 -0.994828314445791 -> 0.040861 0.092713 -0.99485; origin xyz=0.0635994253292133 -0.000590202035316956 -0.0153997469552429 rpy=-1.57079925003102 -1.15568185911555 -0.00927676327375631 -> xyz=0.063599 -0.0005902 -0.0154 rpy=-1.5708 -1.1557 -0.0092768
- joint 3C_joint: axis -0.0348227777562482 -0.994834846523427 -0.0953467476742054 -> -0.034736 -0.99486 -0.09511; origin xyz=0.171099056984165 0 0 rpy=1.57085675367315 2.20692556657909E-05 -0.765289631009453 -> xyz=0.1711 0 0 rpy=1.5709 2.2069E-05 -0.76529
- joint 4A_joint: axis 0 0 0.999999999991391 -> 0 0 1; origin xyz=-0.255974054373996 -1.01206206817619 -0.00588646684487949 rpy=-1.5707963267949 -1.50475510925559 3.14159265358979 -> xyz=-0.25597 -1.0121 -0.0058865 rpy=-1.5708 -1.5048 3.1416
- joint 4B_joint: axis -0.026183695853635 -0.0696804058154778 -0.997225679130273 -> -0.026184 -0.06968 -0.99723; origin xyz=0.0635992616466633 -0.000576968315201321 0.00570022034299766 rpy=-1.57078983356474 -1.21135560970982 -0.00907755888534315 -> xyz=0.063599 -0.00057697 0.0057002 rpy=-1.5708 -1.2114 -0.0090776
- joint 4C_joint: axis 0.0494409591559326 -0.997225674243885 0.055646618824235 -> 0.049441 -0.99723 0.055647; origin xyz=0.171099059852282 0 0 rpy=1.57079637586786 0 -1.08585857681701 -> xyz=0.1711 0 0 rpy=1.5708 0 -1.0859
- joint 5A_joint: axis 0 0 0.999999999991391 -> 0 0 1; origin xyz=-0.136390786035478 -1.01206153239268 -0.0778384850774082 rpy=1.5707963267949 -0.414816831721765 0 -> xyz=-0.13639 -1.0121 -0.077838 rpy=1.5708 -0.41482 0
- joint 5B_joint: axis 0.0311072596905014 0.0951442959394444 -0.99497733710107 -> 0.030965 0.09471 -0.99502; origin xyz=0.0635993103802858 -0.000573903264097668 0.00569993879362163 rpy=-1.57078333798218 -1.25480236320661 -0.00903547312752022 -> xyz=0.063599 -0.0005739 0.0056999 rpy=-1.5708 -1.2548 -0.0090355
- joint 5C_joint: axis 0.0215355717970855 -0.994981619052824 -0.097712828709403 -> 0.021437 -0.99503 -0.097267; origin xyz=0.171078321783105 0 -0.0272330994907475 rpy=1.57083810968274 0 -0.0990644706572842 -> xyz=0.17108 0 -0.027233 rpy=1.5708 0 -0.099064
- joint 6A_joint: axis 0 0 0.999999999991391 -> -0.0039721 -0.039957 0.99919; origin xyz=-0.13991270731822 -1.01206108271275 -0.215549909652052 rpy=1.5707963267949 0.632777255807867 0 -> xyz=-0.13991 -1.0121 -0.21555 rpy=1.5332 0.53367 0.0046181
- joint 6B_joint: axis -0.0995153621342332 0.994932686708951 -0.0143402098102098 -> -0.099515 0.99493 -0.01434; origin xyz=0.0637692737648475 0.0158329936408527 0.00570099857651085 rpy=0 0.143099612060705 3.13252099109131 -> xyz=0.065 0.0092003 0.0063321 rpy=-0.040574 0.14262 3.0276
- joint 6C_joint: axis -0.0505372205435134 -0.99493270384841 -0.0869189516309744 -> -0.0505372205434824 -0.99493270384841 -0.0869189516309928

Commit message: Nuevo ejeA hexapod_description.urdf

File: hexapod_description/urdf/hexapod_description.urdf (robot description, URDF)
Before this commit: robot hexapod_description, 19 links, 18 joints
Links:
- link 1A_link: mass 0.0284343546565839 -> 0.0284343546568847
- link 1B_link: mass 0.0393326462004403 -> 0.0393326462007453
- link 1C_link: mass 0.0544820458081965 -> 0.0544820458081966
- link 2B_link: mass 0.0393326465544562 -> 0.0393326465544563
- link 3A_link: mass 0.0284343550141747 -> 0.0284343550141745
- link 3B_link: mass 0.0393326465589664 -> 0.0393326465589656
- link 3C_link: mass 0.0544820458081965 -> 0.0544820458081966
- link 4A_link: mass 0.0284343546567147 -> 0.0284343546566637
- link 4B_link: mass 0.0393326462005796 -> 0.039332646200528
- link 4C_link: mass 0.0544820458081965 -> 0.0544820458081966
- link 5A_link: mass 0.0284343550237688 -> 0.0284343550237595
- link 5B_link: mass 0.0393326465544563 -> 0.0393326465544561
- link 6B_link: mass 0.039332646558968 -> 0.0393326465589677
- link 6C_link: mass 0.0544820458081965 -> 0.0544820458081966
- link base_link: mass 0.394164283837447 -> 0.394164283837448
Joints:
- joint 1A_joint: axis 0 0 1 -> 0 0 0.999999999991391; origin xyz=-0.26054 -1.0121 -0.28139 rpy=-1.5708 1.4948 -3.1416 -> xyz=-0.260544565013545 -1.01206116241563 -0.281391297394327 rpy=-1.5707963267949 1.49476626971651 -3.14159265358979
- joint 1B_joint: axis -0.044948 -0.050377 -0.99772 -> -0.0449475329048409 -0.0503765997912116 -0.99771835578947; origin xyz=0.06362 -0.00057714 0.005701 rpy=1.5708 0.84229 3.1325 -> xyz=0.0636203974674808 -0.000577139628543943 0.00570103050496762 rpy=1.57080045971871 0.842287346673303 3.13252412666513
- joint 1C_joint: axis -0.010218 -0.99772 -0.066736 -> -0.0102179351135115 -0.997718351691989 -0.0667359310944108; origin xyz=-0.16408 -0.0084589 -0.027239 rpy=1.5708 0 2.2612 -> xyz=-0.164084019172298 -0.00845892892413586 -0.0272391911814598 rpy=1.57079626680283 0 2.26115671183903
- joint 2A_joint: axis 0 0 1 -> 0 0 0.999999999991391; origin xyz=-0.37826 -1.0332 -0.20983 rpy=-1.5708 0.4478 -3.1416 -> xyz=-0.378260308632601 -1.03316169228736 -0.209825331186314 rpy=-1.5707963267949 0.447803456724678 -3.14159265358979
- joint 2B_joint: axis 0.032866 0.05873 -0.99773 -> 0.0328663838674289 0.0587298554671745 -0.997732732192486; origin xyz=0.063599 -0.00057839 -0.0154 rpy=-1.5708 -1.0606 -0.0090858 -> xyz=0.0635994650152483 -0.000578393068543129 -0.0153999472755177 rpy=-1.57080465259821 -1.06059839350069 -0.00908580645889822
- joint 2C_joint: axis 0.061878 0.99773 0.026483 -> 0.0618783699588132 0.997732286459227 0.0264830490707604; origin xyz=0.1711 0 0.0097395 rpy=-1.5708 0 0.6562 -> xyz=0.171099091710239 0 0.00973951247489032 rpy=-1.57079893258156 0 0.656200837708118
- joint 3A_joint: axis 0 0 1 -> 0 0 0.999999999991391; origin xyz=-0.37491 -1.0332 -0.071745 rpy=-1.5708 -0.6336 3.1416 -> xyz=-0.374914944478911 -1.03316214363253 -0.071745054027157 rpy=-1.5707963267949 -0.633602285574073 3.14159265358979
- joint 3B_joint: axis 0.040861 0.092713 -0.99485 -> 0.0408614821447107 0.0927131498264627 -0.994854065240824; origin xyz=0.063599 -0.0005902 -0.0154 rpy=-1.5708 -1.1557 -0.0092768 -> xyz=0.0635994253292133 -0.000590202035316956 -0.0153997469552429 rpy=-1.57079925003102 -1.15568185911555 -0.00927676327375631
- joint 3C_joint: axis -0.034736 -0.99486 -0.09511 -> -0.034736144034017 -0.994860581072829 -0.0951095396113419; origin xyz=0.1711 0 0 rpy=1.5709 2.2069E-05 -0.76529 -> xyz=0.171099056984165 0 0 rpy=1.57085675367315 2.20692556657909E-05 -0.765289631009453
- joint 4A_joint: axis 0 0 1 -> 0 0 0.999999999991391; origin xyz=-0.25597 -1.0121 -0.0058865 rpy=-1.5708 -1.5048 3.1416 -> xyz=-0.255974054373996 -1.01206206817619 -0.00588646684487949 rpy=-1.5707963267949 -1.50475510925559 3.14159265358979
- joint 4B_joint: axis -0.026184 -0.06968 -0.99723 -> -0.0261836958536535 -0.0696804058154684 -0.997225679130273; origin xyz=0.063599 -0.00057697 0.0057002 rpy=-1.5708 -1.2114 -0.0090776 -> xyz=0.0635992616466633 -0.000576968315201321 0.00570022034299766 rpy=-1.57078983356474 -1.21135560970982 -0.00907755888534315
- joint 4C_joint: axis 0.049441 -0.99723 0.055647 -> 0.0494409591558951 -0.997225674243887 0.0556466188242337; origin xyz=0.1711 0 0 rpy=1.5708 0 -1.0859 -> xyz=0.171099059852282 0 0 rpy=1.57079637586786 0 -1.08585857681701
- joint 5A_joint: axis 0 0 1 -> 0 0 0.999999999991391; origin xyz=-0.13639 -1.0121 -0.077838 rpy=1.5708 -0.41482 0 -> xyz=-0.136390786035478 -1.01206153239268 -0.0778384850774082 rpy=1.5707963267949 -0.414816831721765 0
- joint 5B_joint: axis 0.030965 0.09471 -0.99502 -> 0.0310125757403508 0.0948546967313408 -0.995007943010484; origin xyz=0.063599 -0.0005739 0.0056999 rpy=-1.5708 -1.2548 -0.0090355 -> xyz=0.0635993103802858 -0.000573903264097668 0.00569993879362163 rpy=-1.57078333798218 -1.25480236320661 -0.00903547312752022
- joint 5C_joint: axis 0.021437 -0.99503 -0.097267 -> 0.0214699938797235 -0.995012211926078 -0.0974152836097987; origin xyz=0.17108 0 -0.027233 rpy=1.5708 0 -0.099064 -> xyz=0.171078321783105 0 -0.0272330994907475 rpy=1.57083810968274 0 -0.0990644706572842
- joint 6A_joint: axis -0.0039721 -0.039957 0.99919 -> -0.00397209683038318 -0.0399570507149629 0.999193503053804; origin xyz=-0.13991 -1.0121 -0.21555 rpy=1.5332 0.53367 0.0046181 -> xyz=-0.13991270731822 -1.01206108271275 -0.215549909652052 rpy=1.53317914923738 0.533669639617208 0.00461810223899989
- joint 6B_joint: axis -0.099515 0.99493 -0.01434 -> -0.0993712938753993 0.994947385176486 -0.0143194512465494; origin xyz=0.065 0.0092003 0.0063321 rpy=-0.040574 0.14262 3.0276 -> xyz=0.0649997268497639 0.00920026440506977 0.0063321397038929 rpy=-0.0405740891479141 0.142619184593738 3.0275611119679
- joint 6C_joint: axis -0.0505372205434824 -0.99493270384841 -0.0869189516309928 -> -0.0504640578758202 -0.994947402291134 -0.0867931191790598

Commit message: ACTUALIZADO SOLIDWORKS CON EJES DE COORDENADAS CORRECTO en todos los motores

File: hexapod_description/urdf/hexapod_description.urdf (robot description, URDF)
Before this commit: robot hexapod_description, 19 links, 18 joints
Links:
- link 1A_link: mass 0.0284343546568847 -> 0.0263699506975587
- link 1B_link: mass 0.0393326462007453 -> 0.0393326464265752
- link 1C_link: mass 0.0544820458081966 -> 0.0544820458081965
- link 2A_link: mass 0.0284343550237236 -> 0.0263699508381414
- link 2B_link: mass 0.0393326465544563 -> 0.0393326465544565
- link 3A_link: mass 0.0284343550141745 -> 0.0263699508271746
- link 3B_link: mass 0.0393326465589656 -> 0.0393326465562279
- link 4A_link: mass 0.0284343546566637 -> 0.0263699506961657
- link 4B_link: mass 0.039332646200528 -> 0.0393326464252295
- link 5A_link: mass 0.0284343550237595 -> 0.0263699506895398
- link 5B_link: mass 0.0393326465544561 -> 0.0393326465545709
- link 5C_link: mass 0.0544820458081965 -> 0.0544820458081966
- link 6A_link: mass 0.0284343550141806 -> 0.02636995082813
- link 6B_link: mass 0.0393326465589677 -> 0.0393326465581168
- link 6C_link: mass 0.0544820458081966 -> 0.0544820458081965
- link base_link: mass 0.394164283837448 -> 0.406550708950941
Joints:
- joint 1A_joint: axis 0 0 0.999999999991391 -> 0 0.000189825421871335 0.999999981983154; origin xyz=-0.260544565013545 -1.01206116241563 -0.281391297394327 rpy=-1.5707963267949 1.49476626971651 -3.14159265358979 -> xyz=-0.0667468494517693 -0.106777799204074 0.0316495863697956 rpy=0.000187289878885293 0 -2.12946850394786
- joint 1B_joint: axis -0.0449475329048409 -0.0503765997912116 -0.99771835578947 -> -0.0695536721571611 -0.997578192840082 0.000189365704729826; origin xyz=0.0636203974674808 -0.000577139628543943 0.00570103050496762 rpy=1.57080045971871 0.842287346673303 3.13252412666513 -> xyz=0.0752386562540257 -0.00640318117526778 -0.00269755643730618 rpy=0 0 0
- joint 1C_joint: axis -0.0102179351135115 -0.997718351691989 -0.0667359310944108 -> -0.0695536721571234 -0.997578192840085 0.000189365704778719; origin xyz=-0.164084019172298 -0.00845892892413586 -0.0272391911814598 rpy=1.57079626680283 0 2.26115671183903 -> xyz=0.120546165521457 -0.015048025350051 0.120647727640648 rpy=0 0 0
- joint 2A_joint: axis 0 0 0.999999999991391 -> 0 0 0.999999999992758; origin xyz=-0.378260308632601 -1.03316169228736 -0.209825331186314 rpy=-1.5707963267949 0.447803456724678 -3.14159265358979 -> xyz=-0.125845591742144 0.00441551350601397 0.0316500696923352 rpy=0 0 3.10651925204043
- joint 2B_joint: axis 0.0328663838674289 0.0587298554671745 -0.997732732192486 -> 0 -0.999999999992758 0; origin xyz=0.0635994650152483 -0.000578393068543129 -0.0153999472755177 rpy=-1.57080465259821 -1.06059839350069 -0.00908580645889822 -> xyz=0.0755015911121684 -0.00115142974218954 -0.00269876749323283 rpy=0 0 0
- joint 2C_joint: axis 0.0618783699588132 0.997732286459227 0.0264830490707604 -> 0 -0.999999999992758 0; origin xyz=0.171099091710239 0 0.00973951247489032 rpy=-1.57079893258156 0 0.656200837708118 -> xyz=0.12097495075034 -0.00664953949368554 0.121002671452846 rpy=0 0 0
- joint 3A_joint: axis 0 0 0.999999999991391 -> 0 0 0.999999999992459; origin xyz=-0.374914944478911 -1.03316214363253 -0.071745054027157 rpy=-1.5707963267949 -0.633602285574073 3.14159265358979 -> xyz=-0.0590987293485508 0.111193182015965 0.0316504833222655 rpy=0 0 2.05932170084572
- joint 3B_joint: axis 0.0408614821447107 0.0927131498264627 -0.994854065240824 -> -0.227149790678758 -0.973859832101259 0; origin xyz=0.0635994253292133 -0.000590202035316956 -0.0153997469552429 rpy=-1.57079925003102 -1.15568185911555 -0.00927676327375631 -> xyz=0.0732672863787103 -0.0182657395441897 -0.00269870093818958 rpy=0 0 0
- joint 3C_joint: axis -0.034736144034017 -0.994860581072829 -0.0951095396113419 -> -0.227149790678759 -0.973859832101259 0; origin xyz=0.171099056984165 0 0 rpy=1.57085675367315 2.20692556657909E-05 -0.765289631009453 -> xyz=0.0896470917080924 -0.027733299889676 0.143235135491589 rpy=0 0 0
- joint 4A_joint: axis 0 0 0.999999999991391 -> 0 -0.000189825421852773 0.999999981983154; origin xyz=-0.255974054373996 -1.01206206817619 -0.00588646684487949 rpy=-1.5707963267949 -1.50475510925559 3.14159265358979 -> xyz=0.0667468753354276 0.106777537815826 0.0316504136296591 rpy=-0.000187289878885293 0 1.01212414964193
- joint 4B_joint: axis -0.0261836958536535 -0.0696804058154684 -0.997225679130273 -> -0.067341098883768 -0.99772999380135 -0.000189394520411146; origin xyz=0.0635992616466633 -0.000576968315201321 0.00570022034299766 rpy=-1.57078983356474 -1.21135560970982 -0.00907755888534315 -> xyz=0.0752519835596818 -0.00624345785823413 -0.00269995709093918 rpy=0 0 0
- joint 4C_joint: axis 0.0494409591558951 -0.997225674243887 0.0556466188242337 -> -0.0673410988837552 -0.997729993801351 -0.000189394520251638; origin xyz=0.171099059852282 0 0 rpy=1.57079637586786 0 -1.08585857681701 -> xyz=0.120591722612344 -0.0148405749057716 0.120657273965076 rpy=0 0 0
- joint 5A_joint: axis 0 0 0.999999999991391 -> 0 0 0.999999999992758; origin xyz=-0.136390786035478 -1.01206153239268 -0.0778384850774082 rpy=1.5707963267949 -0.414816831721765 0 -> xyz=0.125845617625808 -0.00441577489426207 0.0316499303071216 rpy=0 0 -0.0350734015493665
- joint 5B_joint: axis 0.0310125757403508 0.0948546967313408 -0.995007943010484 -> -0.0658773160112557 -0.997827730232395 0; origin xyz=0.0635993103802858 -0.000573903264097668 0.00569993879362163 rpy=-1.57078333798218 -1.25480236320661 -0.00903547312752022 -> xyz=0.0752608794529679 -0.00613572763718961 -0.00269879522635974 rpy=0 0 0
- joint 5C_joint: axis 0.0214699938797235 -0.995012211926078 -0.0974152836097987 -> -0.0658773160112644 -0.997827730232394 0; origin xyz=0.171078321783105 0 -0.0272330994907475 rpy=1.57083810968274 0 -0.0990644706572842 -> xyz=0.120466525966111 -0.0146350482342145 0.120807379890955 rpy=0 0 0
- joint 6A_joint: axis -0.00397209683038318 -0.0399570507149629 0.999193503053804 -> 0 0 0.999999999992459; origin xyz=-0.13991270731822 -1.01206108271275 -0.215549909652052 rpy=1.53317914923738 0.533669639617208 0.00461810223899989 -> xyz=0.0590987552322091 -0.111193443404212 0.0316495166771902 rpy=0 0 -1.08227095274408
- joint 6B_joint: axis -0.0993712938753993 0.994947385176486 -0.0143194512465494 -> -0.0681438930759001 -0.997675503268196 0; origin xyz=0.0649997268497639 0.00920026440506977 0.0063321397038929 rpy=-0.0405740891479141 0.142619184593738 3.0275611119679 -> xyz=0.0752472515487932 -0.00630076885737318 -0.00269879634505443 rpy=0 0 0
- joint 6C_joint: axis -0.0504640578758202 -0.994947402291134 -0.0867931191790598 -> -0.068143893075898 -0.997675503268196 0; origin xyz=-0.00409101222826194 0.0436501939489914 0.16090715153179 rpy=3.14158945955694 -1.1872473110289 0 -> xyz=0.120933977901671 -0.0149333124138473 0.120302680099782 rpy=0 0 0
